File: PCB/ESP 8266/ESP 8266 .kicad_pcb (KiCad board)
At the start: 2 copper layers, 20 parts

Commit message: update: Update PCB. Create, active gerber files.
Parts:
- removed the Power at (154.9, 43.2)
- removed the Power at (154.9, 57.1)
- added 10k Ohm: 10k Ohm, Resistor_THT:R_Axial_DIN0207_L6.3mm_D2.5mm_P10.16mm_Horizontal, F.Cu at (219.7, 61.0)
- added Sensors pins: Sensors pins, TerminalBlock_Phoenix:TerminalBlock_Phoenix_MKDS-1,5-4-5.08_1x04_P5.08mm_Horizontal, F.Cu at (154.6, 43.2)
- 10k Ohm: renamed from REF**; value R_Axial_DIN0207_L6.3mm_D2.5mm_P10.16mm_Horizontal -> 10k Ohm (x6)
- Relay: renamed from REF**; value PinHeader_1x04_P2.54mm_Vertical -> Relay
- moved 10k Ohm 22.2 mm to (226.1, 86.4), turned to 90 degrees
- moved 10k Ohm 11.4 mm to (241.3, 81.3)
- moved Relay 8.51 mm to (154.9, 68.6), turned to 0 degrees
- moved OLed 126X64 7.63 mm to (190.3, 86.4), turned to 0 degrees
- moved BMP 180 Inside 7.62 mm to (165.1, 86.4), turned to 0 degrees
- moved BMP 180 Outside 7.62 mm to (177.8, 86.4), turned to 0 degrees
- moved 10k Ohm 5.08 mm to (224.8, 67.3)
- moved SWitchs 3.81 mm to (248.9, 47.0)
- moved 10k Ohm 1.27 mm to (241.3, 63.5)
Routing:
- net (no net): track 1241.5 -> 1366.3 mm, vias 3 -> 5
Other:
- board text added: "3 position switchs"
- board text added: "By temo-123 (Github.com)"
- board text added: "Function button"
- board text added: "GND"
- board text added: "RST button"
- board text added: "Res"
- board text added: "Res (GND)"
- board text added: "V 2.2.1"
- board text removed: "3 position button"
- board text removed: "Fun switchs"
- board text removed: "GVD"
- board text removed: "RST switch"
